File: e-track.kicad_sch (KiCad schematic)
At the start: 19 parts, among them J3 Conn_01x06, SW1 SW_Push, SW2 SW_Push, SW3 SW_Push, U1 ESP32-C3-MINI-1, U2 BME280, U5 TPS62842DGR

Commit message: Update PCB design and add SVG exports, improve gitignore
Parts:
- added J1: Batt, Connector_Samtec_MicroPower:Samtec_UMPS-02-XX.X-X-V-S_1x02_P2.0mm_Socket, symbol Connector_Generic:Conn_01x02
Connections:
- net CLK: now also U1.18 (GPIO4/ADC1_CH4); no longer U1.20 (GPIO6)
- net DC: now also U1.20 (GPIO6); no longer U1.18 (GPIO4/ADC1_CH4)
- net DIN: now also U1.16 (GPIO10); no longer U1.21 (GPIO7)
- net RST: now also U1.21 (GPIO7); no longer U1.16 (GPIO10)
- net SCL: now also U1.13 (GPIO1/ADC1_CH1/XTAL_32K_N); no longer U1.12 (GPIO0/ADC1_CH0/XTAL_32K_P)
- net SDA: now also U1.12 (GPIO0/ADC1_CH0/XTAL_32K_P); no longer U1.13 (GPIO1/ADC1_CH1/XTAL_32K_N)
Other:
- note added: "TODO: cargador de bateria"
Changed lines of the file:
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@@
 		(date "2026-05-16")
 	)
+	(text "TODO: cargador de bateria"
+		(exclude_from_sim no)
+		(at 69.85 116.84 0)
+		(effects
+			(font
+				(size 1.27 1.27)
+			)
+		)
+	)
 	(junction
 		(at 66.04 48.26)
@@
 	)
 	(label "CLK"
-		(at 204.47 96.52 180)
+		(at 204.47 91.44 180)
 		(effects
 			(font
@@
 	)
 	(label "SCL"
-		(at 130.81 66.04 0)
+		(at 130.81 68.58 0)
 		(effects
 			(font
@@
 	)
 	(label "SDA"
-		(at 130.81 68.58 0)
+		(at 130.81 66.04 0)
 		(effects
 			(font
@@
 	)
 	(label "RST"
-		(at 204.47 106.68 180)
+		(at 204.47 99.06 180)
 		(effects
 			(font
@@
 	)
 	(label "DIN"
-		(at 204.47 99.06 180)
+		(at 204.47 106.68 180)
 		(effects
 			(font
@@
 	)
 	(label "DC"
-		(at 204.47 91.44 180)
+		(at 204.47 96.52 180)
 		(effects
 			(font
@@
 					(unit 1)
 				)
+			)
+		)
+	)
+	(symbol
+		(lib_id "Connector_Generic:Conn_01x02")
+		(at 33.02 120.65 180)
+		(unit 1)
+		(body_style 1)
+		(exclude_from_sim no)
+		(in_bom yes)
+		(on_board yes)
+		(in_pos_files yes)
+		(dnp no)
+		(fields_autoplaced yes)
+		(property "Reference" "J1"
+			(at 33.02 111.76 0)
+			(show_name no)
+			(do_not_autoplace no)
+			(effects
+				(font
+					(size 1.27 1.27)
+				)
+			)
+		)
+		(property "Value" "Batt"
+			(at 33.02 114.3 0)
+			(show_name no)
+			(do_not_autoplace no)
+			(effects
+				(font
+					(size 1.27 1.27)
+				)
+			)
+		)
+		(property "Footprint" "Connector_Samtec_MicroPower:Samtec_UMPS-02-XX.X-X-V-S_1x02_P2.0mm_Socket"
+			(at 33.02 120.65 0)
+			(hide yes)
+			(show_name no)
+			(do_not_autoplace no)
+			(effects
+				(font
+					(size 1.27 1.27)
+				)
+			)
+		)
+		(property "Datasheet" ""
+			(at 33.02 120.65 0)
+			(hide yes)
+			(show_name no)
+			(do_not_autoplace no)
+			(effects
+				(font
+					(size 1.27 1.27)
+				)
+			)
+		)
+		(property "Description" "Generic connector, single row, 01x02, script generated (kicad-library-utils/schlib/autogen/connector/)"
+			(at 33.02 120.65 0)
+			(hide yes)
+			(show_name no)
+			(do_not_autoplace no)
+			(effects
+				(font
+					(size 1.27 1.27)
+				)
+			)
+		)
+		(property "Part #" ""
+			(at 33.02 120.65 0)
+			(hide yes)
+			(show_name no)
+			(do_not_autoplace no)
+			(effects
+				(font
+					(size 1.27 1.27)
+				)
+			)
+		)
+		(property "Manufacturer" ""
+			(at 33.02 120.65 0)
+			(hide yes)
+			(show_name no)
+			(do_not_autoplace no)
+			(effects
+				(font
+					(size 1.27 1.27)
+				)
+			)
+		)
+		(property "Price" ""
+			(at 33.02 120.65 0)
+			(hide yes)
+			(show_name no)
+			(do_not_autoplace no)
+			(effects
+				(font
+					(size 1.27 1.27)
+				)
+			)
+		)
+		(property "TC" ""
+			(at 33.02 120.65 0)
+			(show_name no)
+			(do_not_autoplace no)
+			(effects
+				(font
+					(size 1.27 1.27)
+				)
+			)
+		)
+		(property "Current" ""
+			(at 33.02 120.65 0)
+			(show_name no)
+			(do_not_autoplace no)
+			(effects
+				(font
+					(size 1.27 1.27)
+				)
+			)
+		)
+		(property "Power" ""
+			(at 33.02 120.65 0)
+			(show_name no)
+			(do_not_autoplace no)
+			(effects
+				(font
+					(size 1.27 1.27)
+				)
+			)
+		)
+		(property "Voltage" ""
+			(at 33.02 120.65 0)
+			(show_name no)
+			(do_not_autoplace no)
+			(effects
+				(font
+					(size 1.27 1.27)
+				)
+			)
+		)
+		(property "Tol" ""
+			(at 33.02 120.65 0)
+			(show_name no)
+			(do_not_autoplace no)
+			(effects
+				(font
+					(size 1.27 1.27)
+				)
+			)
+		)
+		(property "LCSC" ""
+			(at 33.02 120.65 0)
+			(hide yes)
+			(show_name no)
+			(do_not_autoplace no)
+			(effects
+				(font
+					(size 1.27 1.27)
+				)
+			)
+		)
+		(pin "1"
+		)
+		(pin "2"
+		)
+		(instances
+			(project "e-track"
+				(path "/a48d5c3f-2ff7-4ab0-b08d-97b515d567a2"
+					(reference "J1")
+					(unit 1)
+				)

Commit message: agregando conector y RTC
Parts:
- added C17: 100nF, Capacitor_SMD:C_0603_1608Metric, symbol Device:C
- added J4: Conn_01x04, MR-footprint:pogo-pin-female-4P-2.54, symbol Connector_Generic:Conn_01x04
- added U3: PCF8563TS, Package_SO:MSOP-8_3x3mm_P0.65mm, symbol Timer_RTC:PCF8563TS
- added Y1: 32.768kHz, Crystal:Crystal_SMD_3215-2Pin_3.2x1.5mm, symbol Device:Crystal
Connections:
- net +3V3: now also C17.2, U3.8 (VDD)
- net GND: now also C17.1, U3.4 (VSS)
- net SCL: now also U3.6 (SCL)
- net SDA: now also U3.5 (SDA)
- new net: U3.1 (OSCI), Y1.2
- new net: U3.2 (OSCO), Y1.1
- no-connect marks 2 -> 4
Other:
- moved on the sheet: C14, C16, C7, C9, J1, L3, R13, R14, R15, U2, U5
